File: RepeaterActivators.kicad_sch (KiCad schematic)
At the start: 63 parts, among them Q1 2N7000, Q2 2N7000, Q3 2N7000, Q4 2N7000, Q5 2N7000, Q6 2N7000, Q7 2N7000, Q8 2N7000, U1 74LS273, U2 74LS04, U3 74LS138, U4 74LS138, U5 74AHC04, U6 74LS04

Commit message: DBD: v1.0 complete
Parts:
- added J?: Conn_01x02_Female, symbol Connector:Conn_01x02_Female
Connections:
- net GND: now also J?.2 (Pin_2)
- net Radio2 Frequency Down: now reaches J?.3, Q8.3 (D)
- net Radio2 Frequency Up: now reaches J?.4, Q6.3 (D)
- net Radio2 Fan: now reaches Q5.3 (D)
- net Radio2 Fan: now also J?.1 (Pin_1)
Changed lines of the file:
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@@
     (stroke (width 0) (type default) (color 0 0 0 0))
   )
-  (wire (pts (xy 320.04 181.61) (xy 331.47 181.61))
-    (stroke (width 0) (type default) (color 0 0 0 0))
-  )
   (wire (pts (xy 81.28 64.77) (xy 81.28 110.49))
     (stroke (width 0) (type default) (color 0 0 0 0))
@@
     (stroke (width 0) (type default) (color 0 0 0 0))
   )
+  (wire (pts (xy 339.09 147.32) (xy 364.49 147.32))
+    (stroke (width 0) (type default) (color 0 0 0 0))
+  )
   (wire (pts (xy 266.7 73.66) (xy 267.97 73.66))
     (stroke (width 0) (type default) (color 0 0 0 0))
@@
     (stroke (width 0) (type default) (color 0 0 0 0))
   )
+  (wire (pts (xy 363.22 149.86) (xy 364.49 149.86))
+    (stroke (width 0) (type default) (color 0 0 0 0))
+  )
   (wire (pts (xy 285.75 204.47) (xy 334.01 204.47))
     (stroke (width 0) (type default) (color 0 0 0 0))
@@
     (stroke (width 0) (type default) (color 0 0 0 0))
   )
+  (wire (pts (xy 339.09 181.61) (xy 339.09 147.32))
+    (stroke (width 0) (type default) (color 0 0 0 0))
+  )
   (wire (pts (xy 31.75 30.48) (xy 31.75 34.29))
     (stroke (width 0) (type default) (color 0 0 0 0))
@@
     (stroke (width 0) (type default) (color 0 0 0 0))
   )
+  (wire (pts (xy 320.04 181.61) (xy 339.09 181.61))
+    (stroke (width 0) (type default) (color 0 0 0 0))
+  )
   (wire (pts (xy 49.53 185.42) (xy 52.07 185.42))
     (stroke (width 0) (type default) (color 0 0 0 0))
@@
     (effects (font (size 1.27 1.27)) (justify left bottom))
   )
+  (label "Radio2 Fan" (at 347.98 147.32 0)
+    (effects (font (size 1.27 1.27)) (justify left bottom))
+  )
+  (label "Radio2 Frequency Up" (at 355.6 116.84 180)
+    (effects (font (size 1.27 1.27)) (justify right bottom))
+  )
   (label "Radio1 Fan" (at 346.71 68.58 0)
     (effects (font (size 1.27 1.27)) (justify left bottom))
   )
+  (label "Radio2 Frequency Down" (at 355.6 114.3 180)
+    (effects (font (size 1.27 1.27)) (justify right bottom))
+  )
   (label "Radio1 PTT" (at 321.31 48.26 0)
     (effects (font (size 1.27 1.27)) (justify left bottom))
@@
     (pin "2")
   )
+  (symbol (lib_id "power:GND") (at 363.22 149.86 0) (unit 1)
+    (in_bom yes) (on_board yes) (fields_autoplaced)
+    (property "Reference" "#PWR?" (id 0) (at 363.22 156.21 0)
+      (effects (font (size 1.27 1.27)) hide)
+    )
+    (property "Value" "GND" (id 1) (at 363.22 154.3034 0))
+    (property "Footprint" "" (id 2) (at 363.22 149.86 0)
+      (effects (font (size 1.27 1.27)) hide)
+    )
+    (property "Datasheet" "" (id 3) (at 363.22 149.86 0)
+      (effects (font (size 1.27 1.27)) hide)
+    )
+    (pin "1")
+  )
   (symbol (lib_id "power:+5V") (at 40.64 110.49 90) (unit 1)
     (in_bom yes) (on_board yes) (fields_autoplaced)
@@
     (pin "2")
   )
+  (symbol (lib_id "Connector:Conn_01x02_Female") (at 369.57 147.32 0) (unit 1)
+    (in_bom yes) (on_board yes) (fields_autoplaced)
+    (property "Reference" "J?" (id 0) (at 370.2812 147.7553 0)
+      (effects (font (size 1.27 1.27)) (justify left))
+    )
+    (property "Value" "Conn_01x02_Female" (id 1) (at 370.2812 150.2922 0)
+      (effects (font (size 1.27 1.27)) (justify left))
+    )
+    (property "Footprint" "" (id 2) (at 369.57 147.32 0)
+      (effects (font (size 1.27 1.27)) hide)
+    )
+    (property "Datasheet" "~" (id 3) (at 369.57 147.32 0)
+      (effects (font (size 1.27 1.27)) hide)
+    )
+    (pin "1")
+    (pin "2")
+  )
   (symbol (lib_id "74xx:74LS138") (at 161.29 104.14 0) (unit 1)
     (in_bom yes) (on_board yes) (fields_autoplaced)
@@
       (reference "#PWR?") (unit 1) (value "+12V") (footprint "")
     )
+    (path "/a25267b9-ddec-49e1-917a-dbbe131268ab"
+      (reference "#PWR?") (unit 1) (value "GND") (footprint "")
+    )
     (path "/a5bd64f3-5621-4bca-86fd-be957a3b8def"
       (reference "#PWR?") (unit 1) (value "+5V") (footprint "")
@@
       (reference "J?") (unit 1) (value "AudioJack2_Grounded") (footprint "")
     )
+    (path "/e2626fb5-7ddd-4bab-a0fd-92adcd815f88"
+      (reference "J?") (unit 1) (value "Conn_01x02_Female") (footprint "")
+    )
     (path "/cd3d77a4-fb3e-4cb0-99fa-c24b85c4f625"
